File: board/board.kicad_pcb (KiCad board)
At the start: 2 copper layers, 21 x 13 mm, 1 part

Commit message: initial
Parts:
- added C1: 100nF, Capacitor_SMD:C_0603_1608Metric, F.Cu at (150.2, 93.5)
- added C2: 100nF, Capacitor_SMD:C_0603_1608Metric, F.Cu at (147.3, 95.5)
- added J1: 001_I2C, on_edge:on_edge_2x05_device, F.Cu at (140.0, 96.5)
- added J2: 001_I2C, on_edge:on_edge_2x05_host, F.Cu at (161.0, 96.5)
- added U1: LPS25HB, Package_LGA:ST_HLGA-10_2.5x2.5mm_P0.6mm_LayoutBorder3x2y, F.Cu at (150.5, 96.3)
- moved LOGO1 7.07 mm to (149.0, 106.0)
Routing:
- net GND: track 0.00 -> 28.9 mm, vias 0 -> 4
- net /pressure/VDD: track 0.00 -> 28.0 mm, vias 0 -> 1
- net /pressure/INT: track 0.00 -> 23.7 mm, vias 0 -> 2
- net /pressure/SCL: track 0.00 -> 22.6 mm, vias 0 -> 2
- net /pressure/~{CS}: track 0.00 -> 22.3 mm, vias 0 -> 2
- net /pressure/SDA: track 0.00 -> 21.3 mm
- net Net-(J1-Pad8): track 0.00 -> 17.0 mm
- net Net-(J1-Pad10): track 0.00 -> 16.2 mm
Other:
- outline, holes or cut-outs redrawn
